File: PCB/ReelyUsefulPcb-4Blocks.brd (EAGLE design)
At the start: 50 x 86 mm, 28 parts, among them Q1 200mA/50V, U2 TJCTM240, U3 PHOTON_SMD

Commit message: Monior improvements to pcb/schematic names and values.
Parts:
- D10: value (none) -> kptd-3216qbc-d-01
- F1: value PTCSMD -> 1206L200PR
- Q1: value 200mA/50V -> BSS138
Changed lines of the file:
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@@
 <element name="FRAME1" library="SparkFun-Aesthetics" package="CREATIVE_COMMONS" value="FRAME-LETTER" x="2.2" y="-58.3"/>
 <element name="LOGO1" library="SparkFun-Aesthetics" package="OSHW-LOGO-L" value="OSHW-LOGOL" x="25" y="-3" locked="yes"/>
-<element name="D10" library="SparkFun-LED" package="LED-1206-BOTTOM" value="" x="24.9999" y="-3.0325" locked="yes" smashed="yes" rot="MR180">
+<element name="D10" library="SparkFun-LED" package="LED-1206-BOTTOM" value="kptd-3216qbc-d-01" x="24.9999" y="-3.0325" locked="yes" smashed="yes" rot="MR180">
 <attribute name="NAME" x="22.4599" y="-4.3025" size="1.27" layer="26" rot="MR180"/>
 <attribute name="VALUE" x="22.4599" y="-0.4925" size="1.27" layer="28" rot="MR180"/>
+<attribute name="FARNELL" value="2290349" x="24.9999" y="-3.0325" size="1.778" layer="28" rot="MR180" display="off"/>
 </element>
 <element name="D2" library="SparkFun-LED" package="LED3MM" value="PD204-6C" x="21" y="3" locked="yes" smashed="yes" rot="MR180">
@@
 <attribute name="VALUE" x="15.875" y="46.355" size="1.27" layer="27"/>
 </element>
-<element name="Q1" library="SparkFun-DiscreteSemi" package="SOT23-3" value="200mA/50V" x="36.195" y="53.34" smashed="yes">
+<element name="Q1" library="SparkFun-DiscreteSemi" package="SOT23-3" value="BSS138" x="36.195" y="53.34" smashed="yes">
 <attribute name="PROD_ID" value="TRANS-00830" x="36.195" y="53.34" size="1.778" layer="27" display="off"/>
 <attribute name="NAME" x="37.2745" y="54.483" size="0.8128" layer="25"/>
+<attribute name="FARNELL" value="9845330" x="36.195" y="53.34" size="1.778" layer="27" display="off"/>
 </element>
 <element name="R10" library="SparkFun-Resistors" package="1206" value="10R" x="29.21" y="52.705" smashed="yes">
@@
 <attribute name="NAME" x="2.159" y="57.531" size="0.8128" layer="25"/>
 </element>
-<element name="F1" library="SparkFun-PowerIC" package="PTC-1206" value="PTCSMD" x="13.6525" y="56.515" smashed="yes" rot="R270">
+<element name="F1" library="SparkFun-PowerIC" package="PTC-1206" value="1206L200PR" x="13.6525" y="56.515" smashed="yes" rot="R270">
 <attribute name="PROD_ID" value="RES-11150" x="13.6525" y="56.515" size="2.54" layer="27" rot="R270" display="off"/>
 <attribute name="NAME" x="11.176" y="55.5625" size="0.8128" layer="25"/>
+<attribute name="FARNELL" value="2383297" x="13.6525" y="56.515" size="1.778" layer="27" rot="R270" display="off"/>
 </element>
 <element name="R11" library="SparkFun-Resistors" package="1206" value="10k" x="46.355" y="42.8625" smashed="yes" rot="R180">
